File: hardware/Arduino_Nano/Trackuino-v2_Arduino_Nano.kicad_pcb (KiCad board)
At the start: 2 copper layers, 22 parts, among them J1 Conn_Coaxial, P1 Terminal Block x2, SW1 SW_Push_Dual, U1 Radiometrix HX1, U2 GPS, U3 Logic Level Converter - Bi-Di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, U4 OpenLog, U5 LD1117S33TR_SOT223, U6 LD1117S50TR_SOT223, U7 TMP36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

Commit message: finished nano board
Parts:
- moved U5 90.8 mm to (94.0, 124.5)
- moved BZ1 75.0 mm to (68.6, 88.9)
- moved U4 74.7 mm to (78.7, 71.1), turned to 90 degrees
- moved R2 71.0 mm to (132.1, 63.5)
- moved C3 70.7 mm to (94.0, 134.6), turned to -90 degrees
- moved D2 69.5 mm to (144.8, 63.5)
- moved U6 68.1 mm to (81.3, 124.5)
- moved C1 62.7 mm to (78.7, 134.6), turned to -90 degrees
- moved C2 61.2 mm to (86.4, 134.6), turned to -90 degrees
- moved D1 58.1 mm to (144.8, 83.8)
- moved U7 55.6 mm to (116.8, 121.9)
- moved U3 54.3 mm to (86.4, 88.9), turned to 90 degrees
- moved SW1 51.4 mm to (116.8, 94.0), turned to -90 degrees
- moved R3 45.7 mm to (132.1, 73.7)
- moved R1 45.1 mm to (132.1, 83.8)
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Connections:
- A1 pad 19: Net-(A1-Pad19) -> unconnected-(A1-Pad19)
- A1 pad 20: Net-(A1-Pad20) -> unconnected-(A1-Pad20)
- A1 pad 25: unconnected-(A1-Pad25) -> Net-(A1-Pad25)
- A1 pad 26: unconnected-(A1-Pad26) -> Net-(A1-Pad26)
- U7 pad 2: Net-(A1-Pad20) -> Net-(A1-Pad26)
- U8 pad 2: Net-(A1-Pad19) -> Net-(A1-Pad25)
Routing:
- net +5V: track 0.00 -> 215.3 mm, vias 0 -> 1
- net +3.3V: track 0.00 -> 141.2 mm, vias 0 -> 1
- net GND: track 0.00 -> 63.1 mm, vias 0 -> 2
- net Net-(A1-Pad5): track 0.00 -> 61.1 mm
- net Net-(A1-Pad7): track 0.00 -> 54.6 mm
- net Net-(J1-Pad2): track 0.00 -> 50.1 mm, vias 0 -> 1
- net Net-(A1-Pad6): track 0.00 -> 48.0 mm
- net Net-(J1-Pad1): track 0.00 -> 42.3 mm, vias 0 -> 1
- net Net-(A1-Pad8): track 0.00 -> 29.0 mm
- net Net-(A1-Pad9): track 0.00 -> 29.0 mm
- net Net-(A1-Pad25): track 0.00 -> 25.4 mm
- net Net-(A1-Pad26): track 0.00 -> 24.9 mm
- net Net-(C1-Pad1): track 0.00 -> 22.3 mm
- net Net-(A1-Pad12): track 0.00 -> 17.4 mm
- net Net-(A1-Pad3): track 0.00 -> 15.6 mm
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- added copper zone on B.Cu, net GND
Other:
- board outline added: 86.4 x 81.3 mm
