File: hardware/Arduino_Nano/Trackuino-v2_Arduino_Nano.kicad_sch (KiCad schematic)
At the start: 22 parts

Commit message: added custom libraries
Parts:
- P1: renamed from P?; value Terminal_Block -> Terminal Block x2; footprint Trackuino:Terminal Block -> Trackuino:Terminal Block x2; symbol Trackuino:Terminal_Block -> Trackuino:Terminal Block x2
- U7: renamed from U?; footprint (none) -> Trackuino:TMP36
- gave numbers to parts that had none: 20

Commit message: finished nano board
Connections:
- net at A1.19 (A0): no longer U8.2
- net at A1.20 (A1): no longer U7.2 (VOUT)
- net at A1.25 (A6): now also U8.2
- net at A1.26 (A7): now also U7.2 (VOUT)
Other:
- moved on the sheet: U7, U8
Changed lines of the file:
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@@
-    (stroke (width 0) (type default) (color 0 0 0 0))
-  )
-  (wire (pts (xy 186.69 134.62) (xy 186.69 119.38))
     (stroke (width 0) (type default) (color 0 0 0 0))
   )
@@
     (stroke (width 0) (type default) (color 0 0 0 0))
   )
+  (wire (pts (xy 179.07 125.73) (xy 171.45 125.73))
+    (stroke (width 0) (type default) (color 0 0 0 0))
+  )
   (wire (pts (xy 172.72 69.85) (xy 172.72 77.47))
     (stroke (width 0) (type default) (color 0 0 0 0))
@@
     (stroke (width 0) (type default) (color 0 0 0 0))
   )
+  (wire (pts (xy 179.07 134.62) (xy 179.07 125.73))
+    (stroke (width 0) (type default) (color 0 0 0 0))
+  )
   (wire (pts (xy 196.85 86.36) (xy 196.85 93.98))
     (stroke (width 0) (type default) (color 0 0 0 0))
@@
     (stroke (width 0) (type default) (color 0 0 0 0))
   )
+  (wire (pts (xy 161.29 119.38) (xy 168.91 119.38))
+    (stroke (width 0) (type default) (color 0 0 0 0))
+  )
   (wire (pts (xy 200.66 76.2) (xy 186.69 76.2))
     (stroke (width 0) (type default) (color 0 0 0 0))
   )
-  (wire (pts (xy 184.15 119.38) (xy 184.15 144.78))
-    (stroke (width 0) (type default) (color 0 0 0 0))
-  )
   (wire (pts (xy 252.73 64.77) (xy 248.92 64.77))
     (stroke (width 0) (type default) (color 0 0 0 0))
@@
     (stroke (width 0) (type default) (color 0 0 0 0))
   )
-  (wire (pts (xy 191.77 134.62) (xy 186.69 134.62))
-    (stroke (width 0) (type default) (color 0 0 0 0))
-  )
   (wire (pts (xy 248.92 59.69) (xy 248.92 49.53))
     (stroke (width 0) (type default) (color 0 0 0 0))
@@
     (stroke (width 0) (type default) (color 0 0 0 0))
   )
+  (wire (pts (xy 161.29 134.62) (xy 161.29 119.38))
+    (stroke (width 0) (type default) (color 0 0 0 0))
+  )
   (wire (pts (xy 81.28 62.23) (xy 93.98 62.23))
     (stroke (width 0) (type default) (color 0 0 0 0))
@@
     (stroke (width 0) (type default) (color 0 0 0 0))
   )
-  (wire (pts (xy 191.77 140.97) (xy 191.77 134.62))
-    (stroke (width 0) (type default) (color 0 0 0 0))
-  )
   (wire (pts (xy 218.44 83.82) (xy 194.31 83.82))
     (stroke (width 0) (type default) (color 0 0 0 0))
@@
     (stroke (width 0) (type default) (color 0 0 0 0))
   )
-  (wire (pts (xy 203.2 140.97) (xy 191.77 140.97))
-    (stroke (width 0) (type default) (color 0 0 0 0))
-  )
   (wire (pts (xy 201.93 119.38) (xy 201.93 132.08))
     (stroke (width 0) (type default) (color 0 0 0 0))
@@
   )
   (wire (pts (xy 181.61 77.47) (xy 181.61 93.98))
+    (stroke (width 0) (type default) (color 0 0 0 0))
+  )
+  (wire (pts (xy 171.45 125.73) (xy 171.45 119.38))
     (stroke (width 0) (type default) (color 0 0 0 0))
   )
@@
     (effects (font (size 5 5)) (justify left bottom))
   )
-  (symbol (lib_id "power:GND") (at 203.2 143.51 270) (unit 1)
-    (in_bom yes) (on_board yes) (fields_autoplaced)
-    (property "Reference" "#PWR0118" (id 0) (at 196.85 143.51 0)
-      (effects (font (size 1.27 1.27)) hide)
-    )
-    (property "Value" "GND" (id 1) (at 199.39 143.5099 90)
-      (effects (font (size 1.27 1.27)) (justify right))
-    )
-    (property "Footprint" "" (id 2) (at 203.2 143.51 0)
-      (effects (font (size 1.27 1.27)) hide)
-    )
-    (property "Datasheet" "" (id 3) (at 203.2 143.51 0)
+  (symbol (lib_id "power:GND") (at 176.53 134.62 180) (unit 1)
+    (in_bom yes) (on_board yes) (fields_autoplaced)
+    (property "Reference" "#PWR0118" (id 0) (at 176.53 128.27 0)
+      (effects (font (size 1.27 1.27)) hide)
+    )
+    (property "Value" "GND" (id 1) (at 176.5301 130.81 90)
+      (effects (font (size 1.27 1.27)) (justify right))
+    )
+    (property "Footprint" "" (id 2) (at 176.53 134.62 0)
+      (effects (font (size 1.27 1.27)) hide)
+    )
+    (property "Datasheet" "" (id 3) (at 176.53 134.62 0)
       (effects (font (size 1.27 1.27)) hide)
     )
@@
     (pin "1")
   )
-  (symbol (lib_id "Trackuino:Terminal Block x3") (at 213.36 140.97 270) (unit 1)
-    (in_bom yes) (on_board yes) (fields_autoplaced)
-    (property "Reference" "U8" (id 0) (at 212.09 139.6999 90)
-      (effects (font (size 1.27 1.27)) (justify left))
-    )
-    (property "Value" "Terminal Block x3" (id 1) (at 212.09 142.2399 90)
-      (effects (font (size 1.27 1.27)) (justify left))
-    )
-    (property "Footprint" "Trackuino:Terminal Block x3" (id 2) (at 213.36 140.97 0)
-      (effects (font (size 1.27 1.27)) hide)
-    )
-    (property "Datasheet" "" (id 3) (at 213.36 140.97 0)
+  (symbol (lib_id "Trackuino:Terminal Block x3") (at 179.07 144.78 180) (unit 1)
+    (in_bom yes) (on_board yes) (fields_autoplaced)
+    (property "Reference" "U8" (id 0) (at 180.3401 143.51 90)
+      (effects (font (size 1.27 1.27)) (justify left))
+    )
+    (property "Value" "Terminal Block x3" (id 1) (at 177.8001 143.51 90)
+      (effects (font (size 1.27 1.27)) (justify left))
+    )
+    (property "Footprint" "Trackuino:Terminal Block x3" (id 2) (at 179.07 144.78 0)
+      (effects (font (size 1.27 1.27)) hide)
+    )
+    (property "Datasheet" "" (id 3) (at 179.07 144.78 0)
       (effects (font (size 1.27 1.27)) hide)
     )
@@
     (pin "3")
   )
-  (symbol (lib_id "power:GND") (at 181.61 144.78 180) (unit 1)
-    (in_bom yes) (on_board yes) (fields_autoplaced)
-    (property "Reference" "#PWR0120" (id 0) (at 181.61 138.43 0)
-      (effects (font (size 1.27 1.27)) hide)
-    )
-    (property "Value" "GND" (id 1) (at 181.61 139.7 0))
-    (property "Footprint" "" (id 2) (at 181.61 144.78 0)
-      (effects (font (size 1.27 1.27)) hide)
-    )
-    (property "Datasheet" "" (id 3) (at 181.61 144.78 0)
+  (symbol (lib_id "power:GND") (at 158.75 134.62 180) (unit 1)
+    (in_bom yes) (on_board yes) (fields_autoplaced)
+    (property "Reference" "#PWR0120" (id 0) (at 158.75 128.27 0)
+      (effects (font (size 1.27 1.27)) hide)
+    )
+    (property "Value" "GND" (id 1) (at 158.75 129.54 0))
+    (property "Footprint" "" (id 2) (at 158.75 134.62 0)
+      (effects (font (size 1.27 1.27)) hide)
+    )
+    (property "Datasheet" "" (id 3) (at 158.75 134.62 0)
       (effects (font (size 1.27 1.27)) hide)
     )
@@
     (pin "9")
   )
-  (symbol (lib_id "power:+5V") (at 203.2 138.43 90) (unit 1)
-    (in_bom yes) (on_board yes) (fields_autoplaced)
-    (property "Reference" "#PWR0117" (id 0) (at 207.01 138.43 0)
-      (effects (font (size 1.27 1.27)) hide)
-    )
-    (property "Value" "+5V" (id 1) (at 199.39 138.4299 90)
-      (effects (font (size 1.27 1.27)) (justify left))
-    )
-    (property "Footprint" "" (id 2) (at 203.2 138.43 0)
-      (effects (font (size 1.27 1.27)) hide)
-    )
-    (property "Datasheet" "" (id 3) (at 203.2 138.43 0)
+  (symbol (lib_id "power:+5V") (at 181.61 134.62 0) (unit 1)
+    (in_bom yes) (on_board yes) (fields_autoplaced)
+    (property "Reference" "#PWR0117" (id 0) (at 181.61 138.43 0)
+      (effects (font (size 1.27 1.27)) hide)
+    )
+    (property "Value" "+5V" (id 1) (at 181.6101 130.81 90)
+      (effects (font (size 1.27 1.27)) (justify left))
+    )
+    (property "Footprint" "" (id 2) (at 181.61 134.62 0)
+      (effects (font (size 1.27 1.27)) hide)
+    )
+    (property "Datasheet" "" (id 3) (at 181.61 134.62 0)
       (effects (font (size 1.27 1.27)) hide)
     )
@@
     (pin "7")
   )
-  (symbol (lib_id "power:+5V") (at 186.69 144.78 0) (unit 1)
-    (in_bom yes) (on_board yes) (fields_autoplaced)
-    (property "Reference" "#PWR0119" (id 0) (at 186.69 148.59 0)
-      (effects (font (size 1.27 1.27)) hide)
-    )
-    (property "Value" "+5V" (id 1) (at 186.69 139.7 0))
-    (property "Footprint" "" (id 2) (at 186.69 144.78 0)
-      (effects (font (size 1.27 1.27)) hide)
-    )
-    (property "Datasheet" "" (id 3) (at 186.69 144.78 0)
+  (symbol (lib_id "power:+5V") (at 163.83 134.62 0) (unit 1)
+    (in_bom yes) (on_board yes) (fields_autoplaced)
+    (property "Reference" "#PWR0119" (id 0) (at 163.83 138.43 0)
+      (effects (font (size 1.27 1.27)) hide)
+    )
+    (property "Value" "+5V" (id 1) (at 163.83 129.54 0))
+    (property "Footprint" "" (id 2) (at 163.83 134.62 0)
+      (effects (font (size 1.27 1.27)) hide)
+    )
+    (property "Datasheet" "" (id 3) (at 163.83 134.62 0)
       (effects (font (size 1.27 1.27)) hide)
     )
@@
     (pin "1")
   )
-  (symbol (lib_id "Trackuino:TMP36") (at 184.15 153.67 180) (unit 1)
-    (in_bom yes) (on_board yes) (fields_autoplaced)
-    (property "Reference" "U7" (id 0) (at 189.23 147.9355 0)
-      (effects (font (size 1.27 1.27)) (justify right))
-    )
-    (property "Value" "TMP36" (id 1) (at 189.23 150.4755 0)
-      (effects (font (size 1.27 1.27)) (justify right))
-    )
-    (property "Footprint" "Trackuino:TMP36" (id 2) (at 184.15 153.67 0)
-      (effects (font (size 1.27 1.27)) hide)
-    )
-    (property "Datasheet" "" (id 3) (at 184.15 153.67 0)
-      (effects (font (size 1.27 1.27)) hide)
-    )
+  (symbol (lib_id "Trackuino:TMP36") (at 161.29 143.51 180) (unit 1)
+    (in_bom yes) (on_board yes) (fields_autoplaced)
+    (property "Reference" "U7" (id 0) (at 166.37 137.7755 0)
+      (effects (font (size 1.27 1.27)) (justify right))
+    )
+    (property "Value" "TMP36" (id 1) (at 166.37 140.3155 0)
+      (effects (font (size 1.27 1.27)) (justify right))
+    )
+    (property "Footprint" "Trackuino:TMP36" (id 2) (at 161.29 143.51 0)
+      (effects (font (size 1.27 1.27)) hide)
+    )
+    (property "Datasheet" "" (id 3) (at 161.29 143.51 0)
+      (effects (font (size 1.27 1.27)) hide)
+    )
